Commit message: yoloTest model working
ros2 launch conveyorbelt_gazebo testworld.launch.py
ros2 run cv_basics opencv_node

File: IFRA_ConveyorBelt/conveyorbelt_gazebo/urdf/camera.urdf (robot description, URDF)
Before this commit: robot setupcam, 3 links, 2 joints
Joints:
- joint camera_joint: origin xyz=0 0 1.5 rpy=0 1.57 0 -> xyz=0 -6 1 rpy=0 0 1.57

Commit message: camera setup for left belt and right belt object detection
Signed-off-by: rkroshan <rkroshan.1999@gmail.com>

File: IFRA_ConveyorBelt/conveyorbelt_gazebo/urdf/camera.urdf (robot description, URDF)
Before this commit: robot setupcam, 3 links, 2 joints
Links:
- removed link camera_link
- removed link camera_link_optical
- added link left_belt_camera_link, mass 1e-5; collision box size=0.1 0.1 0.1; visual box size=0.1 0.1 0.1
- added link left_belt_camera_link_optical
- added link right_belt_camera_link, mass 1e-5; collision box size=0.1 0.1 0.1; visual box size=0.1 0.1 0.1
- added link right_belt_camera_link_optical
Joints:
- removed joint camera_joint
- removed joint camera_optical_joint
- added joint left_belt_camera_joint: type fixed, parent world, child left_belt_camera_link, origin xyz=0 0 1.4 rpy=0 1.57 0
- added joint left_belt_camera_optical_joint: type fixed, parent left_belt_camera_link, child left_belt_camera_link_optical, origin xyz=0 0 0 rpy=-1.57 0 -1.57
- added joint right_belt_camera_joint: type fixed, parent world, child right_belt_camera_link, origin xyz=0 1 1.4 rpy=0 1.57 0
- added joint right_belt_camera_optical_joint: type fixed, parent right_belt_camera_link, child right_belt_camera_link_optical, origin xyz=0 0 0 rpy=-1.57 0 -1.57
