Commit message: created 2 boxes for red and blue color
Signed-off-by: rkroshan <rkroshan.1999@gmail.com>

File: IFRA_ConveyorBelt/conveyorbelt_gazebo/urdf/box_blue.urdf (robot description, URDF)
Before this commit: robot box, 1 links, 0 joints
Links:
- link box: geometry collision box size=0.15 0.15 0.15; visual box size=0.15 0.15 0.15
